File: PCB/REXCPM_UPS_102.kicad_sch (KiCad schematic)
At the start: 9 parts, among them J2 SM04B, J3 Conn_02x20_Odd_Even, U1 742G02

Commit message: remove all mention of model 200, since REXCPM does not support it
Other:
- title: REXCPM UPS 102_200 -> REXCPM UPS 102
Changed lines of the file:
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@@
   (paper "USLetter")
   (title_block
-    (title "REXCPM UPS 102_200")
-    (date "2023-09-02")
-    (rev "001")
+    (title "REXCPM UPS 102")
+    (date "2023-09-20")
+    (rev "002")
     (company "Brian K. White - b.kenyon.w@gmail.com")
     (comment 1 "Replacement REXCPM system bus interface with memory battery")
@@
     (pin "1")
     (instances
-      (project "REXCPM_UPS_102_200"
+      (project "REXCPM_UPS_102"
         (path "/28a4b045-d480-4410-adb7-fa6b33984079"
           (reference "#PWR03") (unit 1)
@@
     (pin "1")
     (instances
-      (project "REXCPM_UPS_102_200"
+      (project "REXCPM_UPS_102"
         (path "/28a4b045-d480-4410-adb7-fa6b33984079"
           (reference "#PWR08") (unit 1)
@@
     (pin "1")
     (instances
-      (project "REXCPM_UPS_102_200"
+      (project "REXCPM_UPS_102"
         (path "/28a4b045-d480-4410-adb7-fa6b33984079"
           (reference "#PWR018") (unit 1)
@@
     (pin "2")
     (instances
-      (project "REXCPM_UPS_102_200"
+      (project "REXCPM_UPS_102"
         (path "/28a4b045-d480-4410-adb7-fa6b33984079"
           (reference "BT2") (unit 1)
@@
     (pin "1")
     (instances
-      (project "REXCPM_UPS_102_200"
+      (project "REXCPM_UPS_102"
         (path "/28a4b045-d480-4410-adb7-fa6b33984079"
           (reference "#PWR02") (unit 1)
@@
     (pin "1")
     (instances
-      (project "REXCPM_UPS_102_200"
+      (project "REXCPM_UPS_102"
         (path "/28a4b045-d480-4410-adb7-fa6b33984079"
           (reference "#PWR013") (unit 1)
@@
     (pin "8")
     (instances
-      (project "REXCPM_UPS_102_200"
+      (project "REXCPM_UPS_102"
         (path "/28a4b045-d480-4410-adb7-fa6b33984079"
           (reference "U1") (unit 2)
@@
     (pin "1")
     (instances
-      (project "REXCPM_UPS_102_200"
+      (project "REXCPM_UPS_102"
         (path "/28a4b045-d480-4410-adb7-fa6b33984079"
           (reference "#PWR04") (unit 1)
@@
     (pin "1")
     (instances
-      (project "REXCPM_UPS_102_200"
+      (project "REXCPM_UPS_102"
         (path "/28a4b045-d480-4410-adb7-fa6b33984079"
           (reference "#PWR014") (unit 1)
@@
     (pin "1")
     (instances
-      (project "REXCPM_UPS_102_200"
+      (project "REXCPM_UPS_102"
         (path "/28a4b045-d480-4410-adb7-fa6b33984079"
           (reference "#PWR017") (unit 1)
@@
     (pin "MP")
     (instances
-      (project "REXCPM_UPS_102_200"
+      (project "REXCPM_UPS_102"
         (path "/28a4b045-d480-4410-adb7-fa6b33984079"
           (reference "J2") (unit 1)
@@
     (pin "9")
     (instances
-      (project "REXCPM_UPS_102_200"
+      (project "REXCPM_UPS_102"
         (path "/28a4b045-d480-4410-adb7-fa6b33984079"
           (reference "J3") (unit 1)
@@
     (pin "8")
     (instances
-      (project "REXCPM_UPS_102_200"
+      (project "REXCPM_UPS_102"
         (path "/28a4b045-d480-4410-adb7-fa6b33984079"
           (reference "U1") (unit 1)
@@
     (pin "3")
     (instances
-      (project "REXCPM_UPS_102_200"
+      (project "REXCPM_UPS_102"
         (path "/28a4b045-d480-4410-adb7-fa6b33984079"
           (reference "D1") (unit 1)
@@
     (pin "1")
     (instances
-      (project "REXCPM_UPS_102_200"
+      (project "REXCPM_UPS_102"
         (path "/28a4b045-d480-4410-adb7-fa6b33984079"
           (reference "#PWR012") (unit 1)
@@
     (pin "1")
     (instances
-      (project "REXCPM_UPS_102_200"
+      (project "REXCPM_UPS_102"
         (path "/28a4b045-d480-4410-adb7-fa6b33984079"
           (reference "#PWR01") (unit 1)
@@
     (pin "1")
     (instances
-      (project "REXCPM_UPS_102_200"
+      (project "REXCPM_UPS_102"
         (path "/28a4b045-d480-4410-adb7-fa6b33984079"
           (reference "#PWR06") (unit 1)
@@
     (pin "8")
     (instances
-      (project "REXCPM_UPS_102_200"
+      (project "REXCPM_UPS_102"
         (path "/28a4b045-d480-4410-adb7-fa6b33984079"
           (reference "U1") (unit 3)
@@
     (pin "2")
     (instances
-      (project "REXCPM_UPS_102_200"
+      (project "REXCPM_UPS_102"
         (path "/28a4b045-d480-4410-adb7-fa6b33984079"
           (reference "BT1") (unit 1)
@@
     (pin "1")
     (instances
-      (project "REXCPM_UPS_102_200"
+      (project "REXCPM_UPS_102"
         (path "/28a4b045-d480-4410-adb7-fa6b33984079"
           (reference "#PWR015") (unit 1)
@@
     (pin "2")
     (instances
-      (project "REXCPM_UPS_102_200"
+      (project "REXCPM_UPS_102"
         (path "/28a4b045-d480-4410-adb7-fa6b33984079"
           (reference "BT3") (unit 1)
@@
     (pin "1")
     (instances
-      (project "REXCPM_UPS_102_200"
+      (project "REXCPM_UPS_102"
         (path "/28a4b045-d480-4410-adb7-fa6b33984079"
           (reference "#PWR07") (unit 1)
@@
     (pin "1")
     (instances
-      (project "REXCPM_UPS_102_200"
+      (project "REXCPM_UPS_102"
         (path "/28a4b045-d480-4410-adb7-fa6b33984079"
           (reference "#PWR016") (unit 1)
@@
     (pin "2")
     (instances
-      (project "REXCPM_UPS_102_200"
+      (project "REXCPM_UPS_102"
         (path "/28a4b045-d480-4410-adb7-fa6b33984079"
           (reference "C1") (unit 1)
@@
     (pin "1")
     (instances
-      (project "REXCPM_UPS_102_200"
+      (project "REXCPM_UPS_102"
         (path "/28a4b045-d480-4410-adb7-fa6b33984079"
           (reference "#FLG02") (unit 1)
@@
     (pin "1")
     (instances
-      (project "REXCPM_UPS_102_200"
+      (project "REXCPM_UPS_102"
         (path "/28a4b045-d480-4410-adb7-fa6b33984079"
           (reference "#PWR09") (unit 1)
@@
     (pin "1")
     (instances
-      (project "REXCPM_UPS_102_200"
+      (project "REXCPM_UPS_102"
         (path "/28a4b045-d480-4410-adb7-fa6b33984079"
           (reference "#PWR011") (unit 1)
@@
     (pin "1")
     (instances
-      (project "REXCPM_UPS_102_200"
+      (project "REXCPM_UPS_102"
         (path "/28a4b045-d480-4410-adb7-fa6b33984079"
           (reference "#FLG01") (unit 1)
@@
     (pin "1")
     (instances
-      (project "REXCPM_UPS_102_200"
+      (project "REXCPM_UPS_102"
         (path "/28a4b045-d480-4410-adb7-fa6b33984079"
           (reference "#PWR010") (unit 1)
@@
     (pin "1")
     (instances
-      (project "REXCPM_UPS_102_200"
+      (project "REXCPM_UPS_102"
         (path "/28a4b045-d480-4410-adb7-fa6b33984079"
           (reference "#PWR05") (unit 1)
@@
     (pin "2")
     (instances
-      (project "REXCPM_UPS_102_200"
+      (project "REXCPM_UPS_102"
         (path "/28a4b045-d480-4410-adb7-fa6b33984079"
           (reference "BT4") (unit 1)

Commit message: replace BAT54C with BAV170 to protect batteries better
Parts:
- D1: value BAT54C -> BAV170
Changed lines of the file:
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@@
   (title_block
     (title "REXCPM UPS 102")
-    (date "2023-09-20")
-    (rev "002")
+    (date "2023-09-21")
+    (rev "003")
     (company "Brian K. White - b.kenyon.w@gmail.com")
     (comment 1 "Replacement REXCPM system bus interface with memory battery")
@@
       (effects (font (size 1.27 1.27)))
     )
-    (property "Value" "BAT54C" (at 88.9 123.19 0)
+    (property "Value" "BAV170" (at 88.9 123.19 0)
       (effects (font (size 1.27 1.27)))
     )
@@
       (effects (font (size 1.27 1.27)) (justify left) hide)
     )
-    (property "Datasheet" "datasheets/bat54c.pdf" (at 90.932 127 0)
-      (effects (font (size 1.27 1.27)) hide)
-    )
+    (property "Datasheet" "datasheets/BAV170.pdf" (at 90.932 127 0)
+      (effects (font (size 1.27 1.27)) hide)
+    )
